Commit message: Finish Assignment 5

File: manipulator/dummy_gazebo/robot/dummy.xacro (robot description, xacro)
@@ -5,3 +5,6 @@
   <xacro:include filename="$(find ${description_package})/robot/dynamics/robot.xacro"/>
   <xacro:dummy_robot package="${description_package}"/>
+  <!-- TODO 5 : -->
+  <xacro:include filename="$(find ${gazebo_package})/robot/ros2_control.gazebo.xacro"/>
+  <xacro:controller_plugins/>
 </robot>

File: manipulator/dummy_gazebo/robot/ros2_control.gazebo.xacro (robot description, xacro)
@@ -1,3 +1,47 @@
 <?xml version='1.0' encoding='utf-8'?>
 <robot xmlns:xacro="http://www.ros.org/wiki/xacro">
+    <!-- ################################### -->
+    <!-- TODO 5 : Create Controller as Macro -->
+    <!-- ################################### -->
+    <!-- ##########  CODE HERE   ########### -->
+    <!-- ################################### -->
+    <xacro:macro name="controller_plugins" params="">
+        <!-- ROS2 Control -->
+        <ros2_control name="GazeboSystem" type="system">
+            <!-- Create Hardware Interface ( Resource Manager ) - Gazebo -->
+            <hardware>
+                <plugin>gazebo_ros2_control/GazeboSystem</plugin>
+            </hardware>
+            <!-- Macro for joints -->
+            <xacro:macro name="robot_joint" params="link_id">
+                <joint name="joint_${link_id}">
+                    <!-- Command to Hardware Interface -->
+                    <command_interface name="position">
+                        <param name="min"> -3.14 </param>
+                        <param name="max"> +3.14 </param>
+                    </command_interface>
+                    <!-- Readings from Hardware Interface - Position -->
+                    <state_interface name="position">
+                        <param name="initial_value"> 0.0 </param>
+                    </state_interface>
+                    <!-- Readings from Hardware Interface - Velocity -->
+                    <state_interface name="velocity"></state_interface>
+                    <!-- Readings from Hardware Interface - Effort -->
+                    <state_interface name="effort"></state_interface>
+                </joint>
+            </xacro:macro>
+            <!-- LET's CALL the MACRO to Create things -->
+            <xacro:robot_joint link_id="1"/>
+            <xacro:robot_joint link_id="2"/>
+            <xacro:robot_joint link_id="3"/>
+        </ros2_control>
+        <!-- Create gazebo plugin to read above macro and create controller(driver) to joints in gazebo -->
+        <gazebo>
+            <plugin filename="libgazebo_ros2_control.so" name="gazebo_ros2_joint_control">
+                <!-- YAML says that we can control the macro above (joint1, joint2, joint3) -->
+                <parameters>$(find dummy_gazebo)/config/_controller_config.yaml</parameters>
+            </plugin>
+        </gazebo>
+    </xacro:macro>
+    <!-- ################################### -->
 </robot>

Commit message: Finish Assignment 6

File: manipulator/dummy_gazebo/robot/dummy.xacro (robot description, xacro)
@@ -1,10 +1,22 @@
 <?xml version='1.0' encoding='utf-8'?>
 <robot xmlns:xacro="http://www.ros.org/wiki/xacro" name="dummy">
+  <!-- ######################### -->
+  <!-- TODO 6 - Spawn Many Robot -->
+  <!-- ######################### -->
+  <!-- ######## CODE HERE ###### -->
+  <!-- For Getting things from outside -->
+  <xacro:arg name="robot_name" default=""/>
+  <!-- Things from outside to Xacro Variable -->
+  <xacro:property name="namespace" value="$(arg robot_name)"/>
+  <!-- ######################### -->
   <xacro:property name="description_package" value="dummy_description"/>
   <xacro:property name="gazebo_package" value="dummy_gazebo"/>
   <xacro:include filename="$(find ${description_package})/robot/dynamics/robot.xacro"/>
   <xacro:dummy_robot package="${description_package}"/>
-  <!-- TODO 5 : -->
   <xacro:include filename="$(find ${gazebo_package})/robot/ros2_control.gazebo.xacro"/>
-  <xacro:controller_plugins/>
+  <!-- ######################### -->
+  <!-- TODO 6 - Spawn Many Robot -->
+  <!-- ######################### -->
+  <xacro:controller_plugins namespace="${namespace}"/>
+  <!-- ######################### -->
 </robot>

File: manipulator/dummy_gazebo/robot/ros2_control.gazebo.xacro (robot description, xacro)
@@ -2,9 +2,8 @@
 <robot xmlns:xacro="http://www.ros.org/wiki/xacro">
     <!-- ################################### -->
-    <!-- TODO 5 : Create Controller as Macro -->
+    <!-- TODO 6 : Spawn Many Robot -->
     <!-- ################################### -->
-    <!-- ##########  CODE HERE   ########### -->
+    <xacro:macro name="controller_plugins" params="namespace">
     <!-- ################################### -->
-    <xacro:macro name="controller_plugins" params="">
         <!-- ROS2 Control -->
         <ros2_control name="GazeboSystem" type="system">
@@ -39,9 +38,15 @@
         <gazebo>
             <plugin filename="libgazebo_ros2_control.so" name="gazebo_ros2_joint_control">
+                <!-- ################################### -->
+                <!-- TODO 6 : Spawn Many Robot -->
+                <!-- ################################### -->
                 <!-- YAML says that we can control the macro above (joint1, joint2, joint3) -->
-                <parameters>$(find dummy_gazebo)/config/_controller_config.yaml</parameters>
+                <parameters>$(find dummy_gazebo)/config/${namespace}_controller_config.yaml</parameters>
+                <ros>
+                    <namespace>/${namespace}</namespace>
+                </ros>
+                <!-- ################################### -->
             </plugin>
         </gazebo>
     </xacro:macro>
-    <!-- ################################### -->
 </robot>
