Commit message: Finish Assignment 7

File: manipulator/dummy_gazebo/robot/ros2_control.gazebo.xacro (robot description, xacro)
@@ -1,9 +1,5 @@
 <?xml version='1.0' encoding='utf-8'?>
 <robot xmlns:xacro="http://www.ros.org/wiki/xacro">
-    <!-- ################################### -->
-    <!-- TODO 6 : Spawn Many Robot -->
-    <!-- ################################### -->
     <xacro:macro name="controller_plugins" params="namespace">
-    <!-- ################################### -->
         <!-- ROS2 Control -->
         <ros2_control name="GazeboSystem" type="system">
@@ -38,7 +34,4 @@
         <gazebo>
             <plugin filename="libgazebo_ros2_control.so" name="gazebo_ros2_joint_control">
-                <!-- ################################### -->
-                <!-- TODO 6 : Spawn Many Robot -->
-                <!-- ################################### -->
                 <!-- YAML says that we can control the macro above (joint1, joint2, joint3) -->
                 <parameters>$(find dummy_gazebo)/config/${namespace}_controller_config.yaml</parameters>
@@ -46,5 +39,4 @@
                     <namespace>/${namespace}</namespace>
                 </ros>
-                <!-- ################################### -->
             </plugin>
         </gazebo>

File: mobile_robot/xxx_gazebo/robot/ros2_control.gazebo.xacro (robot description, xacro)
@@ -1,3 +1,33 @@
 <?xml version='1.0' encoding='utf-8'?>
 <robot xmlns:xacro="http://www.ros.org/wiki/xacro" name="xxx">
+<!-- ################################### -->
+<!-- TODO 7 : Create Controller for XXX  -->
+<!-- ################################### -->
+<xacro:macro name="controller_plugins" params="namespace">
+    <ros2_control name="GazeboSystem" type="system">
+        <hardware>
+            <plugin>gazebo_ros2_control/GazeboSystem</plugin>
+        </hardware>
+        <!-- MACRO for creating wheel -->
+        <xacro:macro name="robot_wheel" params="joint_name">
+            <joint name="${joint_name}">
+                <command_interface name="velocity"/>
+                <command_interface name="effort"/>
+                <state_interface name="velocity"/>
+                <state_interface name="effort"/>
+            </joint>
+        </xacro:macro>
+        <!-- Create Wheel Controllers Driver (gazebo) -->
+        <xacro:robot_wheel joint_name="left_wheel_joint"/>
+        <xacro:robot_wheel joint_name="right_wheel_joint"/>
+    </ros2_control>
+    <gazebo>
+        <plugin filename="libgazebo_ros2_control.so" name="gazebo_ros2_wheel_control">
+            <parameters>$(find xxx_gazebo)/config/${namespace}_controller_config.yaml</parameters>
+            <ros>
+                <namespace>/${namespace}</namespace>
+            </ros>
+        </plugin>
+    </gazebo>
+</xacro:macro>
 </robot>

File: mobile_robot/xxx_gazebo/robot/xxx.xacro (robot description, xacro)
@@ -1,4 +1,7 @@
 <?xml version='1.0' encoding='utf-8'?>
 <robot xmlns:xacro="http://www.ros.org/wiki/xacro" name="xxx">
+  <!-- TODO 7 : Create Controller -->
+  <xacro:arg name="robot_name" default=""/>
+  <xacro:property name="namespace" value="$(arg robot_name)"/>
   <xacro:include filename="$(find xxx_description)/robot/dynamics/physical_robot.xacro"/>
   <xacro:include filename="$(find xxx_gazebo)/robot/graphics.gazebo.xacro"/>
@@ -7,3 +10,5 @@
   <xacro:physical_robot/>
   <xacro:gazebo_graphics/>
+  <!-- TODO 7 : Create Controller -->
+  <xacro:controller_plugins namespace="${namespace}"/>
 </robot>
